Commit message: changed form of the robot

File: cart_robot_description/urdf/cart_robot.xacro (robot description, xacro)
@@ -4,8 +4,11 @@
   <!-- Constants for robot dimensions -->
   <!-- <xacro:property name="PI" value="3.1415926535897931"/> -->
-  <xacro:property name="mass" value="1" /> <!-- arbitrary value for mass -->
+  <xacro:property name="mass" value="500" /> <!-- arbitrary value for mass -->
+  <xacro:property name="horizontal" value="1" /> <!-- Square dimensions (widthxwidth) of beams -->
+  <xacro:property name="vertical" value="0.5" /> <!-- Square dimensions (widthxwidth) of beams -->
   <xacro:property name="width" value="0.1" /> <!-- Square dimensions (widthxwidth) of beams -->
-  <xacro:property name="height1" value="2" /> <!-- Link 1 -->
-  <xacro:property name="height2" value="1" /> <!-- Link 2 -->
+  <xacro:property name="height1" value="0.2" /> <!-- Link 1 -->
+  <xacro:property name="height2" value="0.4" /> <!-- Link 2 -->
+  <xacro:property name="height3" value="0.5" /> <!-- Link 3 -->
   <xacro:property name="axel_offset" value="0.05" /> <!-- Space btw top of beam and the each joint -->
   <!-- Import all Gazebo-customization elements, including Gazebo colors -->
@@ -19,5 +22,5 @@
       <origin xyz="0 0 ${height1/2}" rpy="0 0 0"/>
       <geometry>
-	<box size="${width} ${width} ${height1}"/>
+	<box size="${horizontal} ${vertical} ${height1}"/>
       </geometry>
     </collision>
@@ -25,5 +28,5 @@
       <origin xyz="0 0 ${height1/2}" rpy="0 0 0"/>
       <geometry>
-	<box size="${width} ${width} ${height1}"/>
+	<box size="${horizontal} ${vertical} ${height1}"/>
       </geometry>
       <material name="orange"/>
@@ -31,15 +34,45 @@
     <inertial>
       <origin xyz="0 0 ${height1/2}" rpy="0 0 0"/>
-      <mass value="${mass}"/>
+      <mass value="${mass * horizontal * vertical * height1}"/>
       <inertia
-	  ixx="${mass / 12.0 * (width*width + height1*height1)}" ixy="0.0" ixz="0.0"
-	  iyy="${mass / 12.0 * (height1*height1 + width*width)}" iyz="0.0"
-	  izz="${mass / 12.0 * (width*width + width*width)}"/>
+	  ixx="${mass * horizontal * vertical * height1 / 12.0 * (vertical*vertical + height1*height1)}" ixy="0.0" ixz="0.0"
+	  iyy="${mass * horizontal * vertical * height1 / 12.0 * (height1*height1 + horizontal*horizontal)}" iyz="0.0"
+	  izz="${mass * horizontal * vertical * height1 / 12.0 * (horizontal*horizontal + vertical*vertical)}"/>
+    </inertial>
+  </link>
+  <joint name="joint0" type="fixed">
+    <parent link="cart_link"/>
+    <child link="attachment_link"/>
+    <origin xyz="0 0 ${height1}" rpy="0 0 0"/>
+    <axis xyz="0 0 1"/>
+  </joint>
+  <!-- Attachment Link -->
+  <link name="attachment_link">
+    <collision>
+      <origin xyz="0 0 ${height2/2}" rpy="0 0 0"/>
+      <geometry>
+	<box size="${width} ${width} ${height2}"/>
+      </geometry>
+    </collision>
+    <visual>
+      <origin xyz="0 0 ${height2/2}" rpy="0 0 0"/>
+      <geometry>
+	<box size="${width} ${width} ${height2}"/>
+      </geometry>
+      <material name="orange"/>
+    </visual>
+    <inertial>
+      <origin xyz="0 0 ${height2/2}" rpy="0 0 0"/>
+      <mass value="${mass * width * width * height2}"/>
+      <inertia
+	  ixx="${mass * width * width * height2 / 12.0 * (width*width + height2*height2)}" ixy="0.0" ixz="0.0"
+	  iyy="${mass * width * width * height2 / 12.0 * (height2*height2 + width*width)}" iyz="0.0"
+	  izz="${mass * width * width * height2 / 12.0 * (width*width + width*width)}"/>
     </inertial>
   </link>
   <joint name="joint1" type="revolute">
-    <parent link="cart_link"/>
+    <parent link="attachment_link"/>
     <child link="camera_mount_link"/>
-    <origin xyz="${width} 0 ${height1 - axel_offset}" rpy="0 0 0"/>
+    <origin xyz="${width} 0 ${height2 - axel_offset}" rpy="0 0 0"/>
     <axis xyz="1 0 0"/>
     <limit effort="8.0" lower="${-M_PI * 1/6}" upper="${M_PI * 1/6}" velocity="0.45"/>
@@ -49,23 +82,23 @@
   <link name="camera_mount_link">
     <collision>
-      <origin xyz="0 0 ${height2/2 - axel_offset}" rpy="0 0 0"/>
+      <origin xyz="0 0 ${height3/2 - axel_offset}" rpy="0 0 0"/>
       <geometry>
-	<box size="${width} ${width} ${height2}"/>
+	<box size="${width} ${width} ${height3}"/>
       </geometry>
     </collision>
     <visual>
-      <origin xyz="0 0 ${height2/2 - axel_offset}" rpy="0 0 0"/>
+      <origin xyz="0 0 ${height3/2 - axel_offset}" rpy="0 0 0"/>
       <geometry>
-	<box size="${width} ${width} ${height2}"/>
+	<box size="${width} ${width} ${height3}"/>
       </geometry>
       <material name="maroon"/>
     </visual>
     <inertial>
-      <origin xyz="0 0 ${height2/2 - axel_offset}" rpy="0 0 0"/>
-      <mass value="${mass}"/>
+      <origin xyz="0 0 ${height3/2 - axel_offset}" rpy="0 0 0"/>
+      <mass value="${mass * width * width * height3}"/>
       <inertia
-	  ixx="${mass / 12.0 * (width*width + height2*height2)}" ixy="0.0" ixz="0.0"
-	  iyy="${mass / 12.0 * (height2*height2 + width*width)}" iyz="0.0"
-	  izz="${mass / 12.0 * (width*width + width*width)}"/>
+	  ixx="${mass * width * width * height3 / 12.0 * (width*width + height3*height3)}" ixy="0.0" ixz="0.0"
+	  iyy="${mass * width * width * height3 / 12.0 * (height3*height3 + width*width)}" iyz="0.0"
+	  izz="${mass * width * width * height3 / 12.0 * (width*width + width*width)}"/>
     </inertial>
   </link>
@@ -81,5 +114,4 @@
   </transmission>
   <!-- camera1 -->
-  <!-- <xacro:xtion xyz="${0.0074381 + 0} 0 ${0.01875 + height2}" rpy="0 0 0" parent="camera_mount_link" id="1" /> -->
-  <xacro:xtion xyz="0.0074361 0 ${0.01875 + height2 - axel_offset}" rpy="0 0 0" parent="camera_mount_link" id="1" />
+  <xacro:xtion xyz="0.0074361 0 ${0.01875 + height3 - axel_offset}" rpy="0 0 0" parent="camera_mount_link" id="1" />
 </robot>

Commit message: add rtabmap simulation files and change world files

File: cart_robot_description/urdf/cart_robot.xacro (robot description, xacro)
@@ -30,5 +30,5 @@
 	<box size="${horizontal} ${vertical} ${height1}"/>
       </geometry>
-      <material name="orange"/>
+      <material name="red"/>
     </visual>
     <inertial>
@@ -60,5 +60,5 @@
 	<box size="${width} ${width} ${height2}"/>
       </geometry>
-      <material name="orange"/>
+      <material name="red"/>
     </visual>
     <inertial>
@@ -92,5 +92,5 @@
 	<box size="${width} ${width} ${height3}"/>
       </geometry>
-      <material name="maroon"/>
+      <material name="blue"/>
     </visual>
     <inertial>

File: cart_robot_description/urdf/config.xacro (robot description, xacro)
@@ -6,4 +6,10 @@
   <material name="black">
     <color rgba="${0/255} ${0/255} ${0/255} 1.0"/>
+  </material>
+  <material name="red">
+    <color rgba="${255/255} ${0/255} ${0/255} 1.0"/>
+  </material>
+  <material name="blue">
+    <color rgba="${0/255} ${0/255} ${255/255} 1.0"/>
   </material>
   <material name="grey">

Commit message: change files for two cameras

File: cart_robot_description/urdf/cart_robot.xacro (robot description, xacro)
@@ -114,4 +114,6 @@
   </transmission>
   <!-- camera1 -->
-  <xacro:xtion xyz="0.0074361 0 ${0.01875 + height3 - axel_offset}" rpy="0 0 0" parent="camera_mount_link" id="1" />
+  <xacro:xtion xyz="0.0074361 0.015 ${0.01875 + height3 - axel_offset}" rpy="0 0 0" parent="camera_mount_link" id="1" link_xyz="0.01 0.097 0.0"/>
+  <!-- camera2 -->
+  <xacro:xtion xyz="0.0074361 -0.015 ${0.01875 + height3 - axel_offset}" rpy="0 0 0" parent="camera_mount_link" id="2" link_xyz="0.01 -0.103 0.0"/>
 </robot>

File: cart_robot_description/urdf/xtion.xacro (robot description, xacro)
@@ -1,17 +1,19 @@
 <?xml version="1.0"?>
 <robot xmlns:xacro="http://www.ros.org/wiki/xacro" name="xtion">
-  <xacro:macro name="xtion" params="xyz rpy parent id">
+  <xacro:macro name="xtion" params="xyz rpy parent id link_xyz">
     <!-- import gazebo definitions -->
     <xacro:include filename="$(find cart_robot_description)/urdf/xtion.gazebo" />
     <xacro:xtion_gazebo id="${id}"/>
-    <joint name="camera${id}_joint" type="fixed">
+    <joint name="camera${id}_joint" type="revolute">
       <axis xyz="0 0 1" />
       <origin xyz="${xyz}" rpy="${rpy}"/>
       <parent link="${parent}"/>
       <child link="camera${id}_link"/>
+      <limit effort="8.0" lower="${-M_PI * 1/2}" upper="${M_PI * 1/2}" velocity="0.45"/>
+    <dynamics damping="0.7"/>
     </joint>
     <link name="camera${id}_link">
       <collision>
-        <origin xyz="-0.01 0.0 0.0" rpy="0 0 0" />
+        <origin xyz="${link_xyz}" rpy="0 0 0" />
         <geometry>
           <box size="0.04 0.18 0.03"/>
@@ -19,5 +21,5 @@
       </collision>
       <visual>
-        <origin xyz="0 0 0" rpy="${M_PI/2.0} 0 ${M_PI/2.0}" />
+        <origin xyz="${link_xyz}" rpy="${M_PI/2.0} 0 ${M_PI/2.0}" />
         <geometry>
           <mesh filename="package://cart_robot_description/mesh/asus_xtion_pro_live.dae" scale="0.001 0.001 0.001"/>
@@ -31,4 +33,14 @@
       </inertial>
     </link>
+    <transmission name="camera_tran${id}">
+      <type>transmission_interface/SimpleTransmission</type>
+      <joint name="camera${id}_joint">
+        <hardwareInterface>hardware_interface/EffortJointInterface</hardwareInterface>
+      </joint>
+      <actuator name="camera_motor${id}">
+        <hardwareInterface>hardware_interface/EffortJointInterface</hardwareInterface>
+        <mechanicalReduction>1</mechanicalReduction>
+      </actuator>
+    </transmission>
   </xacro:macro>
 </robot>

Commit message: change files for two cameras

File: cart_robot_description/urdf/cart_robot.xacro (robot description, xacro)
@@ -17,4 +17,11 @@
   <xacro:include filename="$(find cart_robot_description)/urdf/config.xacro" />
   <xacro:include filename="$(find cart_robot_description)/urdf/xtion.xacro" />
+  <link name="base_link">
+  </link>
+  <joint name="base_fixed" type="fixed">
+    <origin xyz="0 0 0" rpy="0 0 0"/>
+    <parent link="base_link"/>
+    <child link="cart_link"/>
+  </joint>
   <!-- Cart Link -->
   <link name="cart_link">

Commit message: add shake script

File: cart_robot_description/urdf/cart_robot.xacro (robot description, xacro)
@@ -76,5 +76,5 @@
     <origin xyz="${width} 0 ${height2 - axel_offset}" rpy="0 0 0"/>
     <axis xyz="1 0 0"/>
-    <limit effort="8.0" lower="${-M_PI * 1/6}" upper="${M_PI * 1/6}" velocity="0.45"/>
+    <limit effort="60.0" lower="${-M_PI * 1/6}" upper="${M_PI * 1/6}" velocity="0.45"/>
     <dynamics damping="0.7"/>
   </joint>
