Commit message: gather all branch's files to master

File: cart_robot_description/urdf/cart_robot1.xacro (robot description, xacro)
@@ -17,4 +17,11 @@
   <xacro:include filename="$(find cart_robot_description)/urdf/config.xacro" />
   <xacro:include filename="$(find cart_robot_description)/urdf/xtion.xacro" />
+  <link name="base_link">
+  </link>
+  <joint name="base_fixed" type="fixed">
+    <origin xyz="0 0 0" rpy="0 0 0"/>
+    <parent link="base_link"/>
+    <child link="cart_link"/>
+  </joint>
   <!-- Cart Link -->
   <link name="cart_link">
@@ -114,4 +121,4 @@
   </transmission>
   <!-- camera1 -->
-  <xacro:xtion xyz="0.0074361 0 ${0.01875 + height3 - axel_offset}" rpy="0 0 0" parent="camera_mount_link" id="1" />
+  <xacro:xtion xyz="0.0074361 0 ${0.01875 + height3 - axel_offset}" rpy="0 0 0" parent="camera_mount_link" id="1" link_xyz="0 0 0"/>
 </robot>
